Commit message: 第二十四次提交：完成夹爪的bug修改和上车测试

File: src/rm_description/urdf/mechine_arm.urdf (robot description, URDF)
Before this commit: robot rm_description, 13 links, 12 joints
Joints:
- joint joint_gripper_right: limit lower=-0.06 upper=0.0 effort=10 velocity=1.0 -> lower=-0.06 upper=0.06 effort=10 velocity=1.0

Commit message: 第二十六次提交：修改了一点导航的文件，换了radar成livox_frame

File: src/rm_description/urdf/mechine_arm.urdf (robot description, URDF)
Before this commit: robot rm_description, 13 links, 12 joints
Links:
- removed link radar
- added link livox_frame, mass 0.17859; collision mesh filename=package://rm_description/meshes/radar.STL; visual mesh filename=package://rm_description/meshes/radar.STL
Joints:
- removed joint radar_joint
- added joint livox_frame_joint: type fixed, parent base_link, child livox_frame, origin xyz=0.1572 -0.1665 0.0922 rpy=0 0 0
