Commit message: 第三十一次提交：导入新的urdf模型后真机调试正负转向

File: src/rm_description/urdf/arm.xacro (robot description, xacro)
@@ -80,5 +80,5 @@
     <child link="link_2" />
     <axis xyz="0 0 -1" />
-    <limit lower="-2.1" upper="-0.01" effort="40" velocity="1.5" />
+    <limit lower="-2.1" upper="0.01" effort="40" velocity="1.5" />
   </joint>
   <link name="link_3">
@@ -109,5 +109,5 @@
     <child link="link_3" />
     <axis xyz="0 0 1" />
-    <limit lower="0.01" upper="2.65" effort="30" velocity="1.5" />
+    <limit lower="-2.65" upper="0.01" effort="30" velocity="1.5" />
   </joint>
   <link name="link_4">
@@ -133,5 +133,5 @@
     </collision>
   </link>
-  <joint name="Joint_4" type="continuous">
+  <joint name="Joint_4" type="revolute">
     <origin xyz="-0.0245 0.27098 0" rpy="-1.5708 0 0" />
     <parent link="link_3" />

File: src/rm_description/urdf/engineer.ros2_control.xacro (robot description, xacro)
@@ -5,6 +5,6 @@
         <ros2_control name="${name}" type="system">
             <hardware>
-                <!-- By default, set up controllers for simulation. This won't work on real hardware -->
-                <plugin>mock_components/GenericSystem</plugin>
+                <!--<plugin>mock_components/GenericSystem</plugin>-->
+                <plugin>arm_hardware/ArmHardwareInterface</plugin>
             </hardware>
             <joint name="Joint_1">
